File: rohm-BH1900NUX-breakout.kicad_sch (KiCad schematic)
At the start: 11 parts, among them J1 Conn_01x04_Socket, U1 BH1900NUX-TR

Commit message: Layout updated
Parts:
- J1: footprint Connector_JST:JST_SH_SM04B-SRSS-TB_1x04-1MP_P1.00mm_Horizontal -> Riehlhome:JST_SH_SM04B-SRSS-TB_1x04-1MP_P1.00mm_Horizontal
- U1: footprint Rohm_BH1900NUX_ALT:VSON008X2030_ROM-M -> VSON008X2030_ROM
Connections:
- no-connect marks 0 -> 1
Other:
- moved on the sheet: JP1, R2, R3

Commit message: Final schematics and final layout
Parts:
- U1: symbol Rohm_BH1900NUX_ALT:BH1900NUX-TR -> BH1900NUX:BH1900NUX-TR
Other:
- title: Rohm Semiconductor BH1900NUX Breakout Board -> BH1900NUX - Miniature Temperature Sensor
- moved on the sheet: J1, R2, R3
Changed lines of the file:
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@@
 	(paper "A4")
 	(title_block
-		(title "Rohm Semiconductor BH1900NUX Breakout Board")
-		(date "2025-11-09")
-		(rev "0.1")
+		(title "BH1900NUX - Miniature Temperature Sensor")
+		(date "2026-01-13")
+		(rev "1.0")
 	)
 	(junction
@@
 	(wire
 		(pts
-			(xy 156.21 58.42) (xy 156.21 49.53)
+			(xy 107.95 59.69) (xy 107.95 58.42)
+		)
+		(stroke
+			(width 0)
+			(type default)
+		)
+	)
+	(wire
+		(pts
+			(xy 102.87 67.31) (xy 102.87 58.42)
 		)
 		(stroke
@@
 	(wire
 		(pts
-			(xy 158.75 58.42) (xy 158.75 49.53)
+			(xy 105.41 67.31) (xy 105.41 58.42)
 		)
 		(stroke
@@
 		(pts
 			(xy 213.36 87.63) (xy 220.98 87.63)
+		)
+		(stroke
+			(width 0)
+			(type default)
+		)
+	)
+	(wire
+		(pts
+			(xy 110.49 59.69) (xy 110.49 58.42)
 		)
 		(stroke
@@
 	(global_label "SDA"
 		(shape input)
-		(at 201.93 57.15 270)
+		(at 125.73 59.69 270)
 		(fields_autoplaced yes)
 		(effects
@@
 		)
 		(property "Intersheetrefs" "${INTERSHEET_REFS}"
-			(at 201.93 63.7033 90)
+			(at 125.73 66.2433 90)
 			(effects
 				(font
@@
 	(global_label "SCL"
 		(shape input)
-		(at 196.85 57.15 270)
+		(at 120.65 59.69 270)
 		(fields_autoplaced yes)
 		(effects
@@
 		)
 		(property "Intersheetrefs" "${INTERSHEET_REFS}"
-			(at 196.85 63.6428 90)
+			(at 120.65 66.1828 90)
 			(effects
 				(font
@@
 	(global_label "SDA"
 		(shape input)
-		(at 161.29 49.53 270)
+		(at 107.95 59.69 270)
 		(fields_autoplaced yes)
 		(effects
@@
 		)
 		(property "Intersheetrefs" "${INTERSHEET_REFS}"
-			(at 161.29 56.0833 90)
+			(at 107.95 66.2433 90)
 			(effects
 				(font
@@
 	(global_label "SCL"
 		(shape input)
-		(at 163.83 49.53 270)
+		(at 110.49 59.69 270)
 		(fields_autoplaced yes)
 		(effects
@@
 		)
 		(property "Intersheetrefs" "${INTERSHEET_REFS}"
-			(at 163.83 56.0228 90)
+			(at 110.49 66.1828 90)
 			(effects
 				(font
@@
 	(symbol
 		(lib_id "power:+3V3")
-		(at 158.75 58.42 0)
+		(at 105.41 67.31 0)
 		(mirror x)
 		(unit 1)
@@
 		(dnp no)
 		(property "Reference" "#PWR013"
-			(at 158.75 54.61 0)
+			(at 105.41 63.5 0)
 			(effects
 				(font
@@
 		)
 		(property "Value" "+3V3"
-			(at 158.7501 62.23 90)
+			(at 105.4101 71.12 90)
 			(effects
 				(font
@@
 		)
 		(property "Footprint" ""
-			(at 158.75 58.42 0)
+			(at 105.41 67.31 0)
 			(effects
 				(font
@@
 		)
 		(property "Datasheet" ""
-			(at 158.75 58.42 0)
+			(at 105.41 67.31 0)
 			(effects
 				(font
@@
 		)
 		(property "Description" "Power symbol creates a global label with name \"+3V3\""
-			(at 158.75 58.42 0)
+			(at 105.41 67.31 0)
 			(effects
 				(font
@@
 	(symbol
 		(lib_id "Connector:Conn_01x04_Socket")
-		(at 158.75 44.45 90)
+		(at 105.41 53.34 90)
 		(unit 1)
 		(exclude_from_sim no)
@@
 		(dnp no)
 		(property "Reference" "J1"
-			(at 160.274 41.656 90)
+			(at 106.934 50.546 90)
 			(effects
 				(font
@@
 		)
 		(property "Value" "Conn_01x04_Socket"
-			(at 161.798 39.624 90)
+			(at 108.458 48.514 90)
 			(effects
 				(font
@@
 		)
 		(property "Footprint" "Riehlhome:JST_SH_SM04B-SRSS-TB_1x04-1MP_P1.00mm_Horizontal"
-			(at 158.75 44.45 0)
+			(at 105.41 53.34 0)
 			(effects
 				(font
@@
 		)
 		(property "Datasheet" "~"
-			(at 158.75 44.45 0)
+			(at 105.41 53.34 0)
 			(effects
 				(font
@@
 		)
 		(property "Description" "Generic connector, single row, 01x04, script generated"
-			(at 158.75 44.45 0)
+			(at 105.41 53.34 0)
 			(effects
 				(font
@@
 	(symbol
 		(lib_id "Device:R")
-		(at 196.85 53.34 0)
+		(at 120.65 55.88 0)
 		(mirror y)
 		(unit 1)
@@
 		(dnp no)
 		(property "Reference" "R2"
-			(at 194.564 53.34 90)
+			(at 118.364 55.88 90)
 			(effects
 				(font
@@
 		)
 		(property "Value" "3.3k"
-			(at 196.85 53.594 90)
+			(at 120.65 56.134 90)
 			(effects
 				(font
@@
 		)
 		(property "Footprint" "Resistor_SMD:R_01005_0402Metric"
-			(at 198.628 53.34 90)
+			(at 122.428 55.88 90)
 			(effects
 				(font
@@
 		)
 		(property "Datasheet" "~"
-			(at 196.85 53.34 0)
+			(at 120.65 55.88 0)
 			(effects
 				(font
@@
 		)
 		(property "Description" "Resistor"
-			(at 196.85 53.34 0)
+			(at 120.65 55.88 0)
 			(effects
 				(font
@@
 	)
 	(symbol
-		(lib_id "Rohm_BH1900NUX_ALT:BH1900NUX-TR")
+		(lib_id "BH1900NUX:BH1900NUX-TR")
 		(at 132.08 82.55 0)
 		(unit 1)
@@
 		)
 		(property "Footprint" "VSON008X2030_ROM"
-			(at 152.146 75.692 0)
+			(at 153.416 99.314 0)
 			(effects
 				(font
@@
 	(symbol
 		(lib_id "power:+3V3")
-		(at 201.93 49.53 0)
+		(at 125.73 52.07 0)
 		(unit 1)
 		(exclude_from_sim no)
@@
 		(fields_autoplaced yes)
 		(property "Reference" "#PWR019"
-			(at 201.93 53.34 0)
+			(at 125.73 55.88 0)
 			(effects
 				(font
@@
 		)
 		(property "Value" "+3V3"
-			(at 201.9301 45.72 90)
+			(at 125.7301 48.26 90)
 			(effects
 				(font
@@
 		)
 		(property "Footprint" ""
-			(at 201.93 49.53 0)
+			(at 125.73 52.07 0)
 			(effects
 				(font
@@
 		)
 		(property "Datasheet" ""
-			(at 201.93 49.53 0)
+			(at 125.73 52.07 0)
 			(effects
 				(font
@@
 		)
 		(property "Description" "Power symbol creates a global label with name \"+3V3\""
-			(at 201.93 49.53 0)
+			(at 125.73 52.07 0)
 			(effects
 				(font
@@
 	(symbol
 		(lib_id "power:GND")
-		(at 156.21 58.42 0)
+		(at 102.87 67.31 0)
 		(unit 1)
 		(exclude_from_sim no)
@@
 		(dnp no)
 		(property "Reference" "#PWR018"
-			(at 156.21 64.77 0)
+			(at 102.87 73.66 0)
 			(effects
 				(font
@@
 		)
 		(property "Value" "GND"
-			(at 156.2099 62.23 90)
+			(at 102.8699 71.12 90)
 			(effects
 				(font
@@
 		)
 		(property "Footprint" ""
-			(at 156.21 58.42 0)
+			(at 102.87 67.31 0)
 			(effects
 				(font
@@
 		)
 		(property "Datasheet" ""
-			(at 156.21 58.42 0)
+			(at 102.87 67.31 0)
 			(effects
 				(font
@@
 		)
 		(property "Description" "Power symbol creates a global label with name \"GND\" , ground"
-			(at 156.21 58.42 0)
+			(at 102.87 67.31 0)
 			(effects
 				(font
@@
 	(symbol
 		(lib_id "Device:R")
-		(at 201.93 53.34 0)
+		(at 125.73 55.88 0)
 		(mirror y)
 		(unit 1)
@@
 		(dnp no)
 		(property "Reference" "R3"
-			(at 199.644 53.34 90)
+			(at 123.444 55.88 90)
 			(effects
 				(font
@@
 		)
 		(property "Value" "3.3k"
-			(at 201.93 53.594 90)
+			(at 125.73 56.134 90)
 			(effects
 				(font
@@
 		)
 		(property "Footprint" "Resistor_SMD:R_01005_0402Metric"
-			(at 203.708 53.34 90)
+			(at 127.508 55.88 90)
 			(effects
 				(font
@@
 		)
 		(property "Datasheet" "~"
-			(at 201.93 53.34 0)
+			(at 125.73 55.88 0)
 			(effects
 				(font
@@
 		)
 		(property "Description" "Resistor"
-			(at 201.93 53.34 0)
+			(at 125.73 55.88 0)
 			(effects
 				(font
@@
 	(symbol
 		(lib_id "power:+3V3")
-		(at 196.85 49.53 0)
+		(at 120.65 52.07 0)
 		(unit 1)
 		(exclude_from_sim no)
@@
 		(fields_autoplaced yes)
 		(property "Reference" "#PWR016"
-			(at 196.85 53.34 0)
+			(at 120.65 55.88 0)
 			(effects
 				(font
@@
 		)
 		(property "Value" "+3V3"
-			(at 196.8501 45.72 90)
+			(at 120.6501 48.26 90)
 			(effects
 				(font
@@
 		)
 		(property "Footprint" ""
-			(at 196.85 49.53 0)
+			(at 120.65 52.07 0)
 			(effects
 				(font
@@
 		)
 		(property "Datasheet" ""
-			(at 196.85 49.53 0)
+			(at 120.65 52.07 0)
 			(effects
 				(font
@@
 		)
 		(property "Description" "Power symbol creates a global label with name \"+3V3\""
-			(at 196.85 49.53 0)
-			(effects
-				(font
+			(at 120.65 52.07 0)
+			(effects
+				(font
